Commit message: add weeding_robot

File: agri_robot_description/urdf/agri_robot.urdf.xacro (robot description, xacro)
@@ -2,5 +2,6 @@
 <robot xmlns:xacro="http://www.ros.org/wiki/xacro"  name="agri_robot">
   <xacro:include filename="robot_core.xacro"/>
-  <xacro:include filename="gazebo_control.xacro"/>
+  <!--<xacro:include filename="gazebo_control.xacro"/>-->
+  <xacro:include filename="ros2_control.xacro"/>
   <xacro:include filename="camera_control.xacro"/>
   <!--<xacro:include filename="depth_camera_control.xacro"/>-->

File: agri_robot_description/urdf/ros2_control.xacro (robot description, xacro)
@@ -1,2 +1,39 @@
 <?xml version="1.0"?>
 <robot xmlns:xacro="http://www.ros.org/wiki/xacro">
+    <ros2_control name="GazeboSystem" type="system">
+        <hardware>
+            <plugin>gazebo_ros2_control/GazeboSystem</plugin>
+        </hardware>
+        <joint name="Left_wheel_joint">
+            <command_interface name="velocity">
+                <param name="min">-10</param>
+                <param name="max">10</param>
+            </command_interface>
+            <state_interface name="velocity"/>
+            <state_interface name="position"/>
+        </joint>
+        <joint name="Right_wheel_joint">
+            <command_interface name="velocity">
+                <param name="min">-10</param>
+                <param name="max">10</param>
+            </command_interface>
+                <state_interface name="velocity"/>
+                <state_interface name="position"/>
+        </joint>
+    </ros2_control>
+    <gazebo>
+        <plugin name="gazebo_ros2_control" filename="libgazebo_ros2_control.so">
+            <parameters>./src/weeding_robot/config/controller.yaml</parameters>
+        </plugin>
+    </gazebo>
+    <gazebo>
+    <plugin name="gazebo_ros_joint_state_publisher"
+        filename="libgazebo_ros_joint_state_publisher.so">
+        <update_rate>100</update_rate>
+        <joint_name>Base_caster_left_joint</joint_name>
+        <joint_name>Base_caster_right_joint</joint_name>
+        <joint_name>Caster_wheel_left_joint</joint_name>
+        <joint_name>Caster_wheel_right_joint</joint_name>
+    </plugin>
+  </gazebo>
+</robot>
