Commit message: ros2_control

File: agri_robot_description/urdf/ros2_control.xacro (robot description, xacro)
@@ -1,4 +1,5 @@
 <?xml version="1.0"?>
 <robot xmlns:xacro="http://www.ros.org/wiki/xacro">
+<!--
     <ros2_control name="GazeboSystem" type="system">
         <hardware>
@@ -37,3 +38,36 @@
     </plugin>
   </gazebo>
+-->
+    <ros2_control name="AgriRobot" type="system">
+        <hardware>
+            <plugin>diff_drive_robot/DiffRobotHardware</plugin>
+            <param name="left_wheel_name">Left_wheel_joint</param>
+            <param name="right_wheel_name">Right_wheel_joint</param>
+            <param name="loop_rate">30</param>
+            <param name="device">/dev/ttyACM0</param>
+            <param name="baud_rate">57600</param>
+            <param name="timeout_ms">1000</param>
+            <param name="enc_counts_per_rev">3436</param>
+            <param name="pid_p">20</param>
+            <param name="pid_d">12</param>
+            <param name="pid_i">0</param>
+            <param name="pid_o">50</param>
+        </hardware>
+        <joint name="Left_wheel_joint">
+            <command_interface name="velocity">
+                <param name="min">-10</param>
+                <param name="max">10</param>
+            </command_interface>
+            <state_interface name="velocity"/>
+            <state_interface name="position"/>
+        </joint>
+        <joint name="Right_wheel_joint">
+            <command_interface name="velocity">
+                <param name="min">-10</param>
+                <param name="max">10</param>
+            </command_interface>
+                <state_interface name="velocity"/>
+                <state_interface name="position"/>
+        </joint>
+    </ros2_control>
 </robot>

Commit message: fixed ros2_control

File: agri_robot_description/urdf/ros2_control.xacro (robot description, xacro)
@@ -55,19 +55,13 @@
         </hardware>
         <joint name="Left_wheel_joint">
-            <command_interface name="velocity">
-                <param name="min">-10</param>
-                <param name="max">10</param>
-            </command_interface>
+            <command_interface name="velocity"/>
+            <state_interface name="position"/>
             <state_interface name="velocity"/>
+          </joint>
+          <joint name="Right_wheel_joint">
+            <command_interface name="velocity"/>
             <state_interface name="position"/>
-        </joint>
-        <joint name="Right_wheel_joint">
-            <command_interface name="velocity">
-                <param name="min">-10</param>
-                <param name="max">10</param>
-            </command_interface>
-                <state_interface name="velocity"/>
-                <state_interface name="position"/>
-        </joint>
+            <state_interface name="velocity"/>
+          </joint>
     </ros2_control>
 </robot>
