Commit message: added fixed errors

File: agri_robot_description/urdf/camera_control.xacro (robot description, xacro)
@@ -4,5 +4,5 @@
         <parent link="base_link"/>
         <child link="camera_link"/>
-        <origin xyz="0.548 0 0" rpy="0 ${pi/2} 0"/>
+        <origin xyz="0.548 0 0" rpy="0 ${pi/4} 0"/>
     </joint>
     <link name="camera_link">

Commit message: crop row navigation

File: agri_robot_description/urdf/camera_control.xacro (robot description, xacro)
@@ -4,5 +4,5 @@
         <parent link="base_link"/>
         <child link="camera_link"/>
-        <origin xyz="0.548 0 0" rpy="0 ${pi/4} 0"/>
+        <origin xyz="0.548 0 0" rpy="0 ${pi/3} 0"/>
     </joint>
     <link name="camera_link">

Commit message: fixed navigation

File: agri_robot_description/urdf/camera_control.xacro (robot description, xacro)
@@ -4,5 +4,5 @@
         <parent link="base_link"/>
         <child link="camera_link"/>
-        <origin xyz="0.548 0 0" rpy="0 ${pi/3} 0"/>
+        <origin xyz="0.548 0 0" rpy="0 ${pi/2} 0"/>
     </joint>
     <link name="camera_link">

File: agri_robot_description/urdf/ros2_control.xacro (robot description, xacro)
@@ -22,9 +22,4 @@
         </joint>
     </ros2_control>
-    <gazebo>
-        <plugin name="gazebo_ros2_control" filename="libgazebo_ros2_control.so">
-            <parameters>./src/weeding_robot/config/controller.yaml</parameters>
-        </plugin>
-    </gazebo>
     <gazebo>
     <plugin name="gazebo_ros_joint_state_publisher"
@@ -65,3 +60,8 @@
     </ros2_control>
 -->
+    <gazebo>
+        <plugin name="gazebo_ros2_control" filename="libgazebo_ros2_control.so">
+            <parameters>./src/weeding_robot/config/controller.yaml</parameters>
+        </plugin>
+    </gazebo>
 </robot>

Commit message: Navigation

File: agri_robot_description/urdf/camera_control.xacro (robot description, xacro)
@@ -4,5 +4,5 @@
         <parent link="base_link"/>
         <child link="camera_link"/>
-        <origin xyz="0.548 0 0" rpy="0 ${pi/2} 0"/>
+        <origin xyz="0.548 0 0" rpy="0 ${5*(pi/12)} 0"/>
     </joint>
     <link name="camera_link">

File: agri_robot_description/urdf/ros2_control.xacro (robot description, xacro)
@@ -1,4 +1,5 @@
 <?xml version="1.0"?>
 <robot xmlns:xacro="http://www.ros.org/wiki/xacro">
+<!--
     <ros2_control name="GazeboSystem" type="system">
         <hardware>
@@ -22,4 +23,5 @@
         </joint>
     </ros2_control>
+    -->
     <gazebo>
     <plugin name="gazebo_ros_joint_state_publisher"
@@ -32,5 +34,4 @@
     </plugin>
   </gazebo>
-<!--
     <ros2_control name="AgriRobot" type="system">
         <hardware>
@@ -40,10 +41,10 @@
             <param name="loop_rate">30</param>
             <param name="device">/dev/ttyACM0</param>
-            <param name="baud_rate">57600</param>
+            <param name="baud_rate">115200</param>
             <param name="timeout_ms">1000</param>
             <param name="enc_counts_per_rev">1763</param>
             <param name="pid_p">20</param>
-            <param name="pid_d">12</param>
-            <param name="pid_i">0</param>
+            <param name="pid_d">120</param>
+            <param name="pid_i">10</param>
             <param name="pid_o">50</param>
         </hardware>
@@ -59,5 +60,4 @@
           </joint>
     </ros2_control>
--->
     <gazebo>
         <plugin name="gazebo_ros2_control" filename="libgazebo_ros2_control.so">

Commit message: Update README.md

File: agri_robot_description/urdf/camera_control.xacro (robot description, xacro)
@@ -4,5 +4,5 @@
         <parent link="base_link"/>
         <child link="camera_link"/>
-        <origin xyz="0.548 0 0" rpy="0 ${5*(pi/12)} 0"/>
+        <origin xyz="0.548 0 0" rpy="0 ${7*(pi/18)} 0"/>
     </joint>
     <link name="camera_link">
@@ -32,6 +32,6 @@
                 <image>
                     <format>R8G8B8</format>
-                    <width>640</width>
-                    <height>640</height>
+                    <width>800</width>
+                    <height>600</height>
                 </image>
                 <clip>

File: agri_robot_description/urdf/ros2_control.xacro (robot description, xacro)
@@ -1,5 +1,4 @@
 <?xml version="1.0"?>
 <robot xmlns:xacro="http://www.ros.org/wiki/xacro">
-    <!--
     <ros2_control name="GazeboSystem" type="system">
         <hardware>
@@ -23,5 +22,4 @@
         </joint>
     </ros2_control>
-    -->
     <gazebo>
     <plugin name="gazebo_ros_joint_state_publisher"
@@ -34,4 +32,5 @@
     </plugin>
   </gazebo>
+<!--
     <ros2_control name="AgriRobot" type="system">
         <hardware>
@@ -60,4 +59,5 @@
           </joint>
     </ros2_control>
+    -->
     <gazebo>
         <plugin name="gazebo_ros2_control" filename="libgazebo_ros2_control.so">
